Commit message: Add caster wheel

File: urdf/barista_robot_model.urdf (robot description, URDF)
Before this commit: robot cafeteria robots, 8 links, 7 joints
Links:
- added link back_pitch_link, mass 0.2; collision sphere radius=0.0352; visual sphere radius=0.0352
- added link back_roll_link, mass 0.2; collision cylinder length=0.0206 radius=0.0352; visual cylinder length=0.0206 radius=0.0352
- added link back_yaw_link, mass 0.2; collision cylinder length=0.0206 radius=0.0352; visual cylinder length=0.0206 radius=0.0352
- added link front_pitch_link, mass 0.2; collision sphere radius=0.0352; visual sphere radius=0.0352
- added link front_roll_link, mass 0.2; collision cylinder length=0.0206 radius=0.0352; visual cylinder length=0.0206 radius=0.0352
- added link front_yaw_link, mass 0.2; collision cylinder length=0.0206 radius=0.0352; visual cylinder length=0.0206 radius=0.0352
- link cup_holder_tray: mass None -> 1; geometry collision cylinder length=0.09 radius=0.16; visual cylinder length=0.09 radius=0.16
- link laser_link: mass None -> 0.2; geometry collision cylinder length=0.04 radius=0.025; visual mesh filename=package://barista_robot_description/meshes/hokuyo_urg_04lx.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 scale=1 1 1
- link left_standoff_rod: mass None -> 0.2; geometry collision cylinder length=0.220 radius=0.01; visual cylinder length=0.220 radius=0.01
- link left_wheel: mass None -> 0.2; geometry collision cylinder length=0.0206 radius=0.0352; visual cylinder length=0.0206 radius=0.0352
- link main_body: mass None -> 8; geometry collision cylinder length=0.155 radius=0.178; visual cylinder length=0.155 radius=0.178
- link right_standoff_rod: mass None -> 0.2; geometry collision cylinder length=0.220 radius=0.01; visual cylinder length=0.220 radius=0.01
- link right_wheel: mass None -> 0.2; geometry collision cylinder length=0.0206 radius=0.0352; visual cylinder length=0.0206 radius=0.0352
Joints:
- added joint back_pitch_joint: type continuous, parent back_roll_link, child back_pitch_link, origin xyz=0 0 0 rpy=0 0 0, axis 0 1 0, limit effort=1000.0 velocity=100.0
- added joint back_roll_joint: type continuous, parent back_yaw_link, child back_roll_link, origin xyz=0 0 0 rpy=0 0 0, axis 1 0 0, limit effort=1000.0 velocity=100.0
- added joint back_yaw_joint: type continuous, parent main_body, child back_yaw_link, origin xyz=-0.12 0 -0.0775 rpy=0 0 0, axis 0 0 1, limit effort=1000.0 velocity=100.0
- added joint front_pitch_joint: type continuous, parent front_roll_link, child front_pitch_link, origin xyz=0 0 0 rpy=0 0 0, axis 0 1 0, limit effort=1000.0 velocity=100.0
- added joint front_roll_joint: type continuous, parent front_yaw_link, child front_roll_link, origin xyz=0 0 0 rpy=0 0 0, axis 1 0 0, limit effort=1000.0 velocity=100.0
- added joint front_yaw_joint: type continuous, parent main_body, child front_yaw_link, origin xyz=0.12 0 -0.0775 rpy=0 0 0, axis 0 0 1, limit effort=1000.0 velocity=100.0
- joint main_leftwheel_joint: axis (none) -> 0 1 0; limit (none) -> effort=10000 velocity=1000; type fixed -> continuous
- joint main_rightwheel_joint: axis (none) -> 0 1 0; limit (none) -> effort=10000 velocity=1000; type fixed -> continuous

Commit message: Fixed mesh problem and add sensor & motor plugin

File: urdf/barista_robot_model.urdf (robot description, URDF)
Before this commit: robot cafeteria robots, 14 links, 13 joints
Links:
- removed link left_standoff_rod
- removed link right_standoff_rod
- added link left_standoff_rod_1, mass 0.2; collision cylinder length=0.220 radius=0.01; visual cylinder length=0.220 radius=0.01
- added link left_standoff_rod_2, mass 0.2; collision cylinder length=0.220 radius=0.01; visual cylinder length=0.220 radius=0.01
- added link right_standoff_rod_1, mass 0.2; collision cylinder length=0.220 radius=0.01; visual cylinder length=0.220 radius=0.01
- added link right_standoff_rod_2, mass 0.2; collision cylinder length=0.220 radius=0.01; visual cylinder length=0.220 radius=0.01
Joints:
- removed joint main_leftrod_joint
- removed joint main_rightrod_joint
- added joint main_leftrod_joint_1: type fixed, parent main_body, child left_standoff_rod_1, origin xyz=0.04 0.13 0.1875 rpy=0 0 0
- added joint main_leftrod_joint_2: type fixed, parent main_body, child left_standoff_rod_2, origin xyz=-0.04 0.13 0.1875 rpy=0 0 0
- added joint main_rightrod_joint_1: type fixed, parent main_body, child right_standoff_rod_1, origin xyz=0.04 -0.13 0.1875 rpy=0 0 0
- added joint main_rightrod_joint_2: type fixed, parent main_body, child right_standoff_rod_2, origin xyz=-0.04 -0.13 0.1875 rpy=0 0 0
