Commit message: Put macro in the main files

File: xacro/barista_robot_model.urdf.xacro (robot description, xacro)
@@ -5,4 +5,18 @@
 <xacro:include filename="$(find barista_robot_description)/xacro/cup_holder_tray.xacro" />
 <xacro:include filename="$(find barista_robot_description)/xacro/laser_scanner.xacro" />
+  <!-- Wheel Left -->
+    <xacro:wheel wheel_name="left_wheel" />
+  <!-- Wheel Right -->
+    <xacro:wheel wheel_name="right_wheel" />
+  <!-- Standoff Left rod -->
+    <xacro:standoff_rod standoff_rod_name="left_standoff_rod_1" />
+    <xacro:standoff_rod standoff_rod_name="left_standoff_rod_2" />
+  <!-- Standoff Right rod -->
+    <xacro:standoff_rod standoff_rod_name="right_standoff_rod_1" />.
+    <xacro:standoff_rod standoff_rod_name="right_standoff_rod_2" />
+  <!-- cup_holder_tray -->
+    <xacro:cup_holder_tray cup_holder_tray_name="cup_holder_tray" />.
+  <!-- cup_holder_tray -->
+    <xacro:laser_link laser_link_name="laser_link" />.
 <!-- Material -->
     <material name = "red">

File: xacro/cup_holder_tray.xacro (robot description, xacro)
@@ -1,22 +1,24 @@
 <?xml version="1.0"?>
 <robot xmlns:xacro="http://www.ros.org/wiki/xacro" name="my_box_bot">
-    <link name = "cup_holder_tray">
-        <visual>
-            <origin rpy="0 0 0" xyz="0 0 0"/>
-            <geometry>
-                <cylinder radius = "0.16" length = "0.09"/>
-            </geometry>
-            <material name = "red"/>
-        </visual>
-        <collision>
-            <geometry>
-                <cylinder radius = "0.16" length = "0.09"/>
-            </geometry>
-        </collision>
-        <inertial>
-            <mass value="1"/>
-            <origin rpy="0 0 0" xyz="0 0 0"/>
-            <inertia ixx="0.007075" ixy="0" ixz="0" iyy="0.007075" iyz="0" izz="0.0128"/>
-        </inertial>
-    </link>
+    <xacro:macro name="cup_holder_tray" params="cup_holder_tray_name">
+        <link name = "${cup_holder_tray_name}">
+            <visual>
+                <origin rpy="0 0 0" xyz="0 0 0"/>
+                <geometry>
+                    <cylinder radius = "0.16" length = "0.09"/>
+                </geometry>
+                <material name = "red"/>
+            </visual>
+            <collision>
+                <geometry>
+                    <cylinder radius = "0.16" length = "0.09"/>
+                </geometry>
+            </collision>
+            <inertial>
+                <mass value="1"/>
+                <origin rpy="0 0 0" xyz="0 0 0"/>
+                <inertia ixx="0.007075" ixy="0" ixz="0" iyy="0.007075" iyz="0" izz="0.0128"/>
+            </inertial>
+        </link>
+    </xacro:macro>
 </robot>

File: xacro/laser_scanner.xacro (robot description, xacro)
@@ -1,21 +1,23 @@
 <?xml version="1.0"?>
 <robot xmlns:xacro="http://www.ros.org/wiki/xacro" name="my_box_bot">
-    <link name = "laser_link">
-        <visual>
-            <origin rpy="0 0 0" xyz="0 0 0"/>
-            <geometry>
-                <mesh filename="package://barista_robot_description/meshes/hokuyo_urg_04lx.dae" scale = "1 1 1"/>
-            </geometry>
-        </visual>
-        <collision>
-            <geometry>
-                <cylinder radius = "0.025" length = "0.04"/>
-            </geometry>
-        </collision>
-        <inertial>
-            <mass value="0.2"/>
-            <origin rpy="0 0 0" xyz="0 0 0"/>
-            <inertia ixx="0.000058" ixy="0" ixz="0" iyy="0.000058" iyz="0" izz="0.000062"/>
-        </inertial>
-    </link>
+    <xacro:macro name="laser_link" params="laser_link_name">
+        <link name = "${laser_link_name}">
+            <visual>
+                <origin rpy="0 0 0" xyz="0 0 0"/>
+                <geometry>
+                    <mesh filename="package://barista_robot_description/meshes/hokuyo_urg_04lx.dae" scale = "1 1 1"/>
+                </geometry>
+            </visual>
+            <collision>
+                <geometry>
+                    <cylinder radius = "0.025" length = "0.04"/>
+                </geometry>
+            </collision>
+            <inertial>
+                <mass value="0.2"/>
+                <origin rpy="0 0 0" xyz="0 0 0"/>
+                <inertia ixx="0.000058" ixy="0" ixz="0" iyy="0.000058" iyz="0" izz="0.000062"/>
+            </inertial>
+        </link>
+    </xacro:macro>
 </robot>

File: xacro/standoff.xacro (robot description, xacro)
@@ -22,9 +22,3 @@
         </link>
     </xacro:macro>
-  <!-- Standoff Left rod -->
-    <xacro:standoff_rod standoff_rod_name="left_standoff_rod_1" />
-    <xacro:standoff_rod standoff_rod_name="left_standoff_rod_2" />
-  <!-- Standoff Right rod -->
-    <xacro:standoff_rod standoff_rod_name="right_standoff_rod_1" />.
-    <xacro:standoff_rod standoff_rod_name="right_standoff_rod_2" />
 </robot>

File: xacro/wheel.xacro (robot description, xacro)
@@ -30,7 +30,3 @@
         </gazebo>
     </xacro:macro>
-  <!-- Wheel Left -->
-    <xacro:wheel wheel_name="left_wheel" />
-  <!-- Wheel Right -->
-    <xacro:wheel wheel_name="right_wheel" />
 </robot>

Commit message: Add two argument to XACRO file from launch file

File: xacro/barista_robot_model.urdf.xacro (robot description, xacro)
@@ -326,8 +326,11 @@
     </joint>
 <!-- PLUGINS -->
+  <!-- <xacro:arg name="robot_name" default="robot1"/>
+  <xacro:property name = "robot_name" value = "$(arg robot_name)"/> -->
   <!-- JOINT PUBLISHER -->
   <gazebo>
     <plugin name="barstina_bot_joint_state" filename="libgazebo_ros_joint_state_publisher.so">
       <ros>
+          <!-- <namespace>${robot_name}</namespace> -->
           <remapping>~/out:=joint_states</remapping>
       </ros>

Commit message: Add namespace to each topic and publish frame connect to the world

File: xacro/barista_robot_model.urdf.xacro (robot description, xacro)
@@ -326,11 +326,11 @@
     </joint>
 <!-- PLUGINS -->
-  <!-- <xacro:arg name="robot_name" default="robot1"/>
-  <xacro:property name = "robot_name" value = "$(arg robot_name)"/> -->
+  <xacro:arg name="robot_name" default="robot1"/>
+  <xacro:property name = "robot_name" value = "$(arg robot_name)"/>
   <!-- JOINT PUBLISHER -->
   <gazebo>
     <plugin name="barstina_bot_joint_state" filename="libgazebo_ros_joint_state_publisher.so">
       <ros>
-          <!-- <namespace>${robot_name}</namespace> -->
+          <namespace>${robot_name}</namespace>
           <remapping>~/out:=joint_states</remapping>
       </ros>
@@ -349,4 +349,8 @@
   <gazebo>
     <plugin filename="libgazebo_ros_diff_drive.so" name="differential_drive_controller">
+      <ros>
+          <namespace>${robot_name}</namespace>
+          <remapping>~/cmd_vel:=cmd_vel</remapping>
+      </ros>
       <!-- wheels -->
       <left_joint>main_leftwheel_joint</left_joint>
@@ -361,7 +365,6 @@
       <publish_odom>true</publish_odom>
       <publish_odom_tf>true</publish_odom_tf>
-      <command_topic>cmd_vel</command_topic>
-      <odometry_frame>odom</odometry_frame>
-      <robot_base_frame>base_link</robot_base_frame>
+      <odometry_frame>${robot_name}/odom</odometry_frame>
+      <robot_base_frame>${robot_name}/base_link</robot_base_frame>
     </plugin>
   </gazebo>
@@ -391,4 +394,5 @@
                 <plugin name="laser_link" filename="libgazebo_ros_ray_sensor.so">
                 <ros>
+                    <namespace>${robot_name}</namespace>
                     <remapping>~/out:=scan</remapping>
                 </ros>

Commit message: Add the different color for rick and morty

File: xacro/barista_robot_model.urdf.xacro (robot description, xacro)
@@ -5,4 +5,6 @@
 <xacro:include filename="$(find barista_robot_description)/xacro/cup_holder_tray.xacro" />
 <xacro:include filename="$(find barista_robot_description)/xacro/laser_scanner.xacro" />
+<xacro:arg name="robot_color" default="Red"/>
+<xacro:property name = "robot_color" value = "$(arg robot_color)"/>
   <!-- Wheel Left -->
     <xacro:wheel wheel_name="left_wheel" />
@@ -20,5 +22,5 @@
     <xacro:laser_link laser_link_name="laser_link" />.
 <!-- Material -->
-    <material name = "red">
+    <material name = "Red">
         <color rgba = "1 0 0 0.8 "/>
     </material>
@@ -26,5 +28,5 @@
         <color rgba = "1 1 1 1 "/>
     </material>
-    <material name = "blue">
+    <material name = "Blue">
         <color rgba = "0 0 0.9 0.8 "/>
     </material>
@@ -33,5 +35,5 @@
     </material>
     <gazebo reference="main_body">
-        <material>Gazebo/Red</material>
+        <material>Gazebo/${robot_color}</material>
     </gazebo>
     <gazebo reference="front_yaw_link">
@@ -60,5 +62,5 @@
     </gazebo>
     <gazebo reference="cup_holder_tray">
-        <material>Gazebo/Red</material>
+        <material>Gazebo/${robot_color}</material>
     </gazebo>
     <gazebo reference="laser_link">
@@ -73,5 +75,5 @@
                 <cylinder radius = "0.178" length = "0.155"/>
             </geometry>
-            <material name = "red"/>
+            <material name = "${robot_color}"/>
         </visual>
         <collision>
@@ -115,5 +117,5 @@
             <cylinder radius = "0.0352" length = "0.0206"/>
         </geometry>
-        <material name = "blue"/>
+        <material name = "Blue"/>
       </visual>
       <collision>
@@ -143,5 +145,5 @@
             <cylinder radius = "0.0352" length = "0.0206"/>
         </geometry>
-        <material name = "red"/>
+        <material name = "Red"/>
       </visual>
       <collision>
@@ -207,5 +209,5 @@
             <cylinder radius = "0.0352" length = "0.0206"/>
         </geometry>
-        <material name = "blue"/>
+        <material name = "Blue"/>
       </visual>
       <collision>
@@ -235,5 +237,5 @@
             <cylinder radius = "0.0352" length = "0.0206"/>
         </geometry>
-        <material name = "red"/>
+        <material name = "Red"/>
       </visual>
       <collision>

File: xacro/cup_holder_tray.xacro (robot description, xacro)
@@ -8,5 +8,5 @@
                     <cylinder radius = "0.16" length = "0.09"/>
                 </geometry>
-                <material name = "red"/>
+                <material name = "${robot_color}"/>
             </visual>
             <collision>

Commit message: Fixed robot move slow problem - set all caster wheel link mu to 0

File: xacro/barista_robot_model.urdf.xacro (robot description, xacro)
@@ -187,11 +187,19 @@
     </inertial>
   </link>
-  <gazebo reference="front_pitch_link">
-    <kp>1000000000000000000000000000.0</kp>
-    <kd>1000000000000000000000000000.0</kd>
-    <mu1>0.5</mu1>
-    <mu2>0.5</mu2>
-    <material>Gazebo/Black</material>
-  </gazebo>
+    <gazebo reference="front_pitch_link">
+        <mu1>0.0</mu1>
+        <mu2>0.0</mu2>
+        <material>Gazebo/Black</material>
+    </gazebo>
+    <gazebo reference="front_yaw_link">
+        <mu1>0.0</mu1>
+        <mu2>0.0</mu2>
+        <material>Gazebo/Black</material>
+    </gazebo>
+    <gazebo reference="front_roll_link">
+        <mu1>0.0</mu1>
+        <mu2>0.0</mu2>
+        <material>Gazebo/Black</material>
+    </gazebo>
   <joint name="front_pitch_joint" type="continuous">
     <origin rpy="0 0 0" xyz="0 0 0" />
@@ -279,11 +287,19 @@
     </inertial>
   </link>
-  <gazebo reference="back_pitch_link">
-    <kp>1000000000000000000000000000.0</kp>
-    <kd>1000000000000000000000000000.0</kd>
-    <mu1>0.5</mu1>
-    <mu2>0.5</mu2>
-    <material>Gazebo/Black</material>
-  </gazebo>
+    <gazebo reference="back_pitch_link">
+        <mu1>0.0</mu1>
+        <mu2>0.0</mu2>
+        <material>Gazebo/Black</material>
+    </gazebo>
+    <gazebo reference="back_yaw_link">
+        <mu1>0.0</mu1>
+        <mu2>0.0</mu2>
+        <material>Gazebo/Black</material>
+    </gazebo>
+    <gazebo reference="back_roll_link">
+        <mu1>0.0</mu1>
+        <mu2>0.0</mu2>
+        <material>Gazebo/Black</material>
+    </gazebo>
   <joint name="back_pitch_joint" type="continuous">
     <origin rpy="0 0 0" xyz="0 0 0" />

File: xacro/wheel.xacro (robot description, xacro)
@@ -25,6 +25,6 @@
             <kp>1000000000000000000000000000.0</kp>
             <kd>1000000000000000000000000000.0</kd>
-            <mu1>10.0</mu1>
-            <mu2>10.0</mu2>
+            <mu1>1</mu1>
+            <mu2>1</mu2>
             <material>Gazebo/Black</material>
         </gazebo>
